File: bakeneko-65-pcb.sch (KiCad schematic (older format))
At the start: 161 parts, among them J1 JST SH 4-pin, J2 AVR-ISP-6, SW1 Reset, U1 USBLC6-2SC6, U2 ATmega32U4-AU, Y1 16MHz

Commit message: Update PCB
Connections:
- net D+: now also U1.3 (I/O2); no longer U1.1 (I/O1)
- net D-: now also U1.1 (I/O1); no longer U1.3 (I/O2)
- net at U1.4 (I/O2): now also R2.2; no longer R3.2
- net at U1.6 (I/O1): now also R3.2; no longer R2.2
Other:
- moved on the sheet: U1
Changed lines of the file:
@@
-$EndComp
-$Comp
-L Power_Protection:USBLC6-2SC6 U1
-U 1 1 5F25444E
-P 1350 6500
-F 0 "U1" V 700 6450 50  0000 L CNN
-F 1 "USBLC6-2SC6" V 800 6250 50  0000 L CNN
-F 2 "Package_TO_SOT_SMD:SOT-23-6" H 1350 6000 50  0001 C CNN
-F 3 "https://www.st.com/resource/en/datasheet/usblc6-2.pdf" H 1550 6850 50  0001 C CNN
-F 4 "C7519" H 1350 6500 50  0001 C CNN "LCSC Part #"
-	1    1350 6500
-	0    1    1    0
 $EndComp
 $Comp
 L power:GND #PWR018
 U 1 1 5F256D2D
-P 950 6500
-F 0 "#PWR018" H 950 6250 50  0001 C CNN
-F 1 "GND" V 955 6372 50  0000 R CNN
-F 2 "" H 950 6500 50  0001 C CNN
-F 3 "" H 950 6500 50  0001 C CNN
-	1    950  6500
+P 1450 6050
+F 0 "#PWR018" H 1450 5800 50  0001 C CNN
+F 1 "GND" V 1455 5922 50  0000 R CNN
+F 2 "" H 1450 6050 50  0001 C CNN
+F 3 "" H 1450 6050 50  0001 C CNN
+	1    1450 6050
 	0    1    1    0
 $EndComp
@@
 	0    1    1    0
 $EndComp
-Wire Wire Line
-	2750 6450 2100 6450
-Wire Wire Line
-	2100 6450 2100 6100
-Wire Wire Line
-	2100 6100 1450 6100
-Wire Wire Line
-	2750 6550 2100 6550
-Wire Wire Line
-	2100 6550 2100 6900
-Wire Wire Line
-	2100 6900 1450 6900
 $Comp
 L power:VBUS #PWR08
@@
 L power:VBUS #PWR019
 U 1 1 5F276E32
-P 1750 6500
-F 0 "#PWR019" H 1750 6350 50  0001 C CNN
-F 1 "VBUS" V 1765 6628 50  0000 L CNN
-F 2 "" H 1750 6500 50  0001 C CNN
-F 3 "" H 1750 6500 50  0001 C CNN
-	1    1750 6500
-	0    1    1    0
+P 1450 6850
+F 0 "#PWR019" H 1450 6700 50  0001 C CNN
+F 1 "VBUS" V 1465 6978 50  0000 L CNN
+F 2 "" H 1450 6850 50  0001 C CNN
+F 3 "" H 1450 6850 50  0001 C CNN
+	1    1450 6850
+	0    -1   -1   0
 $EndComp
 $Comp
@@
 	1    0    0    -1
 $EndComp
-Text GLabel 850  6100 0    50   Input ~ 0
+Text GLabel 1050 6350 0    50   Input ~ 0
 D+
-Text GLabel 850  6900 0    50   Input ~ 0
+Text GLabel 1850 6350 2    50   Input ~ 0
 D-
-Wire Wire Line
-	850  6100 1250 6100
-Wire Wire Line
-	1250 6900 850  6900
 $Comp
 L Switch:SW_Push SW1
@@
 	12100 8850 12000 8850
 Connection ~ 12000 8850
+$Comp
+L Power_Protection:USBLC6-2SC6 U1
+U 1 1 5F25444E
+P 1450 6450
+F 0 "U1" H 1400 7000 50  0000 L CNN
+F 1 "USBLC6-2SC6" H 1200 7100 50  0000 L CNN
+F 2 "Package_TO_SOT_SMD:SOT-23-6" H 1450 5950 50  0001 C CNN
+F 3 "https://www.st.com/resource/en/datasheet/usblc6-2.pdf" H 1650 6800 50  0001 C CNN
+F 4 "C7519" H 1450 6450 50  0001 C CNN "LCSC Part #"
+	1    1450 6450
+	-1   0    0    1
+$EndComp
+Wire Wire Line
+	1850 6550 2750 6550
+Wire Wire Line
+	1050 6550 850  6550
+Wire Wire Line
+	850  6550 850  5950
+Wire Wire Line
+	850  5950 2050 5950
+Wire Wire Line
+	2050 5950 2050 6450
+Wire Wire Line
+	2050 6450 2750 6450
 $EndSCHEMATC

Commit message: Update PCB
Parts:
- removed C4: 0.1u, Capacitor_SMD:C_0805_2012Metric, symbol Device:C
- C4: renamed from C5; value 4.7u -> 10u; LCSC Part # C1779 -> C15850
- renumbered C6 to C5, C7 to C6, C8 to C7
Connections:
- net COL0: now also U2.41 (PF0); no longer U2.39 (PF4)
- net COL1: now also U2.8 (PB0); no longer U2.36 (PF7)
- net COL10: no longer U2.26 (PD6)
- net COL11: no longer U2.25 (PD4)
- net COL12: no longer U2.22 (PD5)
- net COL13: no longer U2.21 (PD3)
- net COL14: no longer U2.20 (PD2)
- net COL15: no longer U2.19 (PD1)
- net COL2: no longer U2.38 (PF5)
- net COL3: no longer U2.37 (PF6)
- net COL4: no longer U2.32 (PC7)
- net COL5: no longer U2.31 (PC6)
- net COL6: no longer U2.30 (PB6)
- net COL7: no longer U2.29 (PB5)
- net COL8: no longer U2.28 (PB4)
- net COL9: no longer U2.27 (PD7)
- net MISO: no longer D46.1 (K), D47.1 (K), D48.1 (K), D49.1 (K), D50.1 (K), D51.1 (K), D52.1 (K), D53.1 (K), D54.1 (K), D55.1 (K), D56.1 (K), D57.1 (K), D58.1 (K), D59.1 (K)
- net MOSI: no longer D32.1 (K), D33.1 (K), D34.1 (K), D35.1 (K), D36.1 (K), D37.1 (K), D38.1 (K), D39.1 (K), D40.1 (K), D41.1 (K), D42.1 (K), D43.1 (K), D44.1 (K), D45.1 (K)
- net ROW0: now also U2.1 (PE6); no longer U2.8 (PB0)
- net ROW1: now also U2.12 (PB7); no longer J2.3 (SCK), U2.9 (PB1)
- net ROW4: no longer U2.12 (PB7)
- new net ROW2: D32.1 (K), D33.1 (K), D34.1 (K), D35.1 (K), D36.1 (K), D37.1 (K), D38.1 (K), D39.1 (K), D40.1 (K), D41.1 (K), D42.1 (K), D43.1 (K), D44.1 (K), D45.1 (K)
- new net ROW3: D46.1 (K), D47.1 (K), D48.1 (K), D49.1 (K), D50.1 (K), D51.1 (K), D52.1 (K), D53.1 (K), D54.1 (K), D55.1 (K), D56.1 (K), D57.1 (K), D58.1 (K), D59.1 (K)
- new net SCK: J2.3 (SCK), U2.9 (PB1)
Other:
- moved on the sheet: C4, MX18
Changed lines of the file:
@@
 $Comp
 L Device:C C4
-U 1 1 5F24DABA
+U 1 1 5F24DC72
 P 6300 1750
 F 0 "C4" H 6415 1796 50  0000 L CNN
-F 1 "0.1u" H 6415 1705 50  0000 L CNN
+F 1 "10u" H 6415 1705 50  0000 L CNN
 F 2 "Capacitor_SMD:C_0805_2012Metric" H 6338 1600 50  0001 C CNN
 F 3 "~" H 6300 1750 50  0001 C CNN
-F 4 "C49678" H 6300 1750 50  0001 C CNN "LCSC Part #"
+F 4 "C15850" H 6300 1750 50  0001 C CNN "LCSC Part #"
 	1    6300 1750
 	1    0    0    -1
 $EndComp
-$Comp
-L Device:C C5
-U 1 1 5F24DC72
-P 6700 1750
-F 0 "C5" H 6815 1796 50  0000 L CNN
-F 1 "4.7u" H 6815 1705 50  0000 L CNN
-F 2 "Capacitor_SMD:C_0805_2012Metric" H 6738 1600 50  0001 C CNN
-F 3 "~" H 6700 1750 50  0001 C CNN
-F 4 "C1779" H 6700 1750 50  0001 C CNN "LCSC Part #"
-	1    6700 1750
-	1    0    0    -1
-$EndComp
 Wire Wire Line
 	5100 1350 5100 1450
 Wire Wire Line
 	5100 1450 5500 1450
-Wire Wire Line
-	6700 1450 6700 1600
 Connection ~ 5100 1450
 Wire Wire Line
@@
 Wire Wire Line
 	5100 2050 5500 2050
-Wire Wire Line
-	6700 2050 6700 1900
 Connection ~ 5100 2050
 Wire Wire Line
 	5100 2050 5100 2200
 Wire Wire Line
-	6300 1900 6300 2050
-Connection ~ 6300 2050
-Wire Wire Line
-	6300 2050 6700 2050
-Wire Wire Line
 	5900 1900 5900 2050
-Connection ~ 5900 2050
-Wire Wire Line
-	5900 2050 6300 2050
 Wire Wire Line
 	5500 1900 5500 2050
@@
 Wire Wire Line
 	5900 1600 5900 1450
-Connection ~ 5900 1450
-Wire Wire Line
-	5900 1450 6300 1450
-Wire Wire Line
-	6300 1600 6300 1450
-Connection ~ 6300 1450
-Wire Wire Line
-	6300 1450 6700 1450
 $Comp
 L Device:Polyfuse F1
@@
 $EndComp
 $Comp
-L power:GND #PWR018
+L power:GND #PWR017
 U 1 1 5F256D2D
 P 1450 6050
-F 0 "#PWR018" H 1450 5800 50  0001 C CNN
+F 0 "#PWR017" H 1450 5800 50  0001 C CNN
 F 1 "GND" V 1455 5922 50  0000 R CNN
 F 2 "" H 1450 6050 50  0001 C CNN
@@
 $EndComp
 $Comp
-L power:VBUS #PWR019
+L power:VBUS #PWR020
 U 1 1 5F276E32
 P 1450 6850
-F 0 "#PWR019" H 1450 6700 50  0001 C CNN
+F 0 "#PWR020" H 1450 6700 50  0001 C CNN
 F 1 "VBUS" V 1465 6978 50  0000 L CNN
 F 2 "" H 1450 6850 50  0001 C CNN
@@
 NoConn ~ 3050 6050
 $Comp
-L power:VCC #PWR017
+L power:VCC #PWR018
 U 1 1 5F28483D
 P 3050 6250
-F 0 "#PWR017" H 3050 6100 50  0001 C CNN
+F 0 "#PWR018" H 3050 6100 50  0001 C CNN
 F 1 "VCC" V 3065 6377 50  0000 L CNN
 F 2 "" H 3050 6250 50  0001 C CNN
@@
 $EndComp
 $Comp
-L Device:C C8
+L Device:C C7
 U 1 1 5F284FC4
 P 2650 6750
-F 0 "C8" V 2800 6750 50  0000 C CNN
+F 0 "C7" V 2800 6750 50  0000 C CNN
 F 1 "1u" V 2900 6750 50  0000 C CNN
 F 2 "Capacitor_SMD:C_0805_2012Metric" H 2688 6600 50  0001 C CNN
@@
 $EndComp
 $Comp
-L power:GND #PWR020
+L power:GND #PWR019
 U 1 1 5F286A59
 P 2500 6750
-F 0 "#PWR020" H 2500 6500 50  0001 C CNN
+F 0 "#PWR019" H 2500 6500 50  0001 C CNN
 F 1 "GND" V 2505 6622 50  0000 R CNN
 F 2 "" H 2500 6750 50  0001 C CNN
@@
 XTAL2
 $Comp
-L Device:C C6
+L Device:C C5
 U 1 1 5F297A61
 P 3000 3200
-F 0 "C6" V 2748 3200 50  0000 C CNN
+F 0 "C5" V 2748 3200 50  0000 C CNN
 F 1 "22p" V 2839 3200 50  0000 C CNN
 F 2 "Capacitor_SMD:C_0805_2012Metric" H 3038 3050 50  0001 C CNN
@@
 $EndComp
 $Comp
-L Device:C C7
+L Device:C C6
 U 1 1 5F2984ED
 P 3000 3850
-F 0 "C7" V 2748 3850 50  0000 C CNN
+F 0 "C6" V 2748 3850 50  0000 C CNN
 F 1 "22p" V 2839 3850 50  0000 C CNN
 F 2 "Capacitor_SMD:C_0805_2012Metric" H 3038 3700 50  0001 C CNN
@@
 F 3 "~" H 6850 6750 50  0001 C CNN
 	1    6850 6750
-	1    0    0    -1
+	1    0    0    1
 $EndComp
 $Comp
@@
 Text GLabel 6650 5450 2    50   Input ~ 0
 COL0
-Text GLabel 4250 6750 2    50   Input ~ 0
+Text GLabel 4700 7150 2    50   Input ~ 0
 COL15
-Text GLabel 4250 6850 2    50   Input ~ 0
+Text GLabel 4650 6850 2    50   Input ~ 0
 COL14
-Text GLabel 4250 6950 2    50   Input ~ 0
+Text GLabel 4600 6950 2    50   Input ~ 0
 COL13
-Text GLabel 4250 7150 2    50   Input ~ 0
+Text GLabel 4400 7150 2    50   Input ~ 0
 COL12
-Text GLabel 4250 7050 2    50   Input ~ 0
+Text GLabel 4700 7000 2    50   Input ~ 0
 COL11
-Text GLabel 4250 7250 2    50   Input ~ 0
+Text GLabel 4400 7250 2    50   Input ~ 0
 COL10
-Text GLabel 4250 7350 2    50   Input ~ 0
+Text GLabel 4350 7350 2    50   Input ~ 0
 COL9
-Text GLabel 4250 5850 2    50   Input ~ 0
+Text GLabel 4700 5900 2    50   Input ~ 0
 COL8
-Text GLabel 4250 5950 2    50   Input ~ 0
+Text GLabel 4800 6050 2    50   Input ~ 0
 COL7
-Text GLabel 4250 6050 2    50   Input ~ 0
+Text GLabel 4850 6150 2    50   Input ~ 0
 COL6
-Text GLabel 4250 6350 2    50   Input ~ 0
+Text GLabel 4650 6350 2    50   Input ~ 0
 COL5
-Text GLabel 4250 6450 2    50   Input ~ 0
+Text GLabel 4450 6450 2    50   Input ~ 0
 COL4
-Text GLabel 4250 8250 2    50   Input ~ 0
+Text GLabel 4700 8450 2    50   Input ~ 0
 COL3
-Text GLabel 4250 8150 2    50   Input ~ 0
+Text GLabel 4650 8250 2    50   Input ~ 0
 COL2
-Text GLabel 4250 8350 2    50   Input ~ 0
+Text GLabel 4250 5450 2    50   Input ~ 0
 COL1
-Text GLabel 4250 8050 2    50   Input ~ 0
+Text GLabel 4250 7850 2    50   Input ~ 0
 COL0
-Text GLabel 4250 5450 2    50   Input ~ 0
-ROW0
-Text GLabel 4850 5550 2    50   Input ~ 0
+Text GLabel 4250 6150 2    50   Input ~ 0
 ROW1
-Text GLabel 4850 5650 2    50   Input ~ 0
+Text GLabel 4800 6750 2    50   Input ~ 0
 ROW2
-Text GLabel 4850 5750 2    50   Input ~ 0
+Text GLabel 4700 8000 2    50   Input ~ 0
 ROW3
-Text GLabel 4250 6150 2    50   Input ~ 0
+Text GLabel 4600 7850 2    50   Input ~ 0
 ROW4
-Text GLabel 4850 5550 0    50   Input ~ 0
-SCK
-Text GLabel 4850 5650 0    50   Input ~ 0
-MOSI
-Text GLabel 4850 5750 0    50   Input ~ 0
-MISO
 Wire Wire Line
 	13100 7750 14200 7750
@@
 Wire Wire Line
 	2050 6450 2750 6450
+Text GLabel 4250 7650 2    50   Input ~ 0
+ROW0
+Wire Wire Line
+	6300 1600 6300 1450
+Wire Wire Line
+	6300 1450 5900 1450
+Connection ~ 5900 1450
+Wire Wire Line
+	5900 2050 6300 2050
+Wire Wire Line
+	6300 2050 6300 1900
+Connection ~ 5900 2050
 $EndSCHEMATC

Commit message: Update PCB
Connections:
- net COL0: now also U2.36 (PF7); no longer U2.41 (PF0)
- net COL10: now also U2.25 (PD4)
- net COL11: now also U2.22 (PD5)
- net COL12: now also U2.21 (PD3)
- net COL13: now also U2.20 (PD2)
- net COL14: now also U2.19 (PD1)
- net COL15: now also U2.18 (PD0)
- net COL2: now also U2.39 (PF4)
- net COL3: now also U2.32 (PC7)
- net COL4: now also U2.31 (PC6)
- net COL5: now also U2.30 (PB6)
- net COL6: now also U2.29 (PB5)
- net COL7: now also U2.28 (PB4)
- net COL8: now also U2.27 (PD7)
- net COL9: now also U2.26 (PD6)
- net ROW2: now also U2.37 (PF6)
- net ROW3: now also U2.38 (PF5)
- net ROW4: now also U2.40 (PF1)
- no-connect marks 1 -> 2
Changed lines of the file:
@@
-$EndComp
-$Comp
-L Switch:SW_SPST MX5
-U 1 1 5F2C356D
-P 9050 6050
-F 0 "MX5" H 9050 6285 50  0000 C CNN
-F 1 "1u" H 9050 6194 50  0000 C CNN
-F 2 "Button_Switch_Keyboard:SW_Cherry_MX_1.00u_PCB" H 9050 6050 50  0001 C CNN
-F 3 "~" H 9050 6050 50  0001 C CNN
-	1    9050 6050
-	1    0    0    -1
 $EndComp
 $Comp
@@
 Text GLabel 6650 5450 2    50   Input ~ 0
 COL0
-Text GLabel 4700 7150 2    50   Input ~ 0
+Text GLabel 4250 6650 2    50   Input ~ 0
 COL15
-Text GLabel 4650 6850 2    50   Input ~ 0
+Text GLabel 4250 6750 2    50   Input ~ 0
 COL14
-Text GLabel 4600 6950 2    50   Input ~ 0
+Text GLabel 4250 6850 2    50   Input ~ 0
 COL13
-Text GLabel 4400 7150 2    50   Input ~ 0
+Text GLabel 4250 6950 2    50   Input ~ 0
 COL12
-Text GLabel 4700 7000 2    50   Input ~ 0
+Text GLabel 4250 7150 2    50   Input ~ 0
 COL11
-Text GLabel 4400 7250 2    50   Input ~ 0
+Text GLabel 4250 7050 2    50   Input ~ 0
 COL10
-Text GLabel 4350 7350 2    50   Input ~ 0
+Text GLabel 4250 7250 2    50   Input ~ 0
 COL9
-Text GLabel 4700 5900 2    50   Input ~ 0
+Text GLabel 4250 7350 2    50   Input ~ 0
 COL8
-Text GLabel 4800 6050 2    50   Input ~ 0
+Text GLabel 4250 5850 2    50   Input ~ 0
 COL7
-Text GLabel 4850 6150 2    50   Input ~ 0
+Text GLabel 4250 5950 2    50   Input ~ 0
 COL6
-Text GLabel 4650 6350 2    50   Input ~ 0
+Text GLabel 4250 6050 2    50   Input ~ 0
 COL5
-Text GLabel 4450 6450 2    50   Input ~ 0
+Text GLabel 4250 6350 2    50   Input ~ 0
 COL4
-Text GLabel 4700 8450 2    50   Input ~ 0
-COL3
-Text GLabel 4650 8250 2    50   Input ~ 0
+Text GLabel 4250 8050 2    50   Input ~ 0
 COL2
 Text GLabel 4250 5450 2    50   Input ~ 0
 COL1
-Text GLabel 4250 7850 2    50   Input ~ 0
+Text GLabel 4250 8350 2    50   Input ~ 0
 COL0
 Text GLabel 4250 6150 2    50   Input ~ 0
 ROW1
-Text GLabel 4800 6750 2    50   Input ~ 0
+Text GLabel 4250 8250 2    50   Input ~ 0
 ROW2
-Text GLabel 4700 8000 2    50   Input ~ 0
+Text GLabel 4250 8150 2    50   Input ~ 0
 ROW3
-Text GLabel 4600 7850 2    50   Input ~ 0
+Text GLabel 4250 7950 2    50   Input ~ 0
 ROW4
 Wire Wire Line
@@
 	6300 2050 6300 1900
 Connection ~ 5900 2050
+$Comp
+L Switch:SW_SPST MX5
+U 1 1 5F2C356D
+P 9050 6050
+F 0 "MX5" H 9050 6285 50  0000 C CNN
+F 1 "1u" H 9050 6194 50  0000 C CNN
+F 2 "Button_Switch_Keyboard:SW_Cherry_MX_1.00u_PCB" H 9050 6050 50  0001 C CNN
+F 3 "~" H 9050 6050 50  0001 C CNN
+	1    9050 6050
+	1    0    0    -1
+$EndComp
+Text GLabel 4250 6450 2    50   Input ~ 0
+COL3
+NoConn ~ 4250 7850
 $EndSCHEMATC
