File: bakeneko-65-pcb.sch (KiCad schematic (older format))
At the start: 160 parts, among them J1 JST SH 4-pin, J2 AVR-ISP-6, SW1 Reset, U1 USBLC6-2SC6, U2 ATmega32U4-AU, Y1 16MHz

Commit message: Update PCB
Parts:
- MX65: footprint bakeneko-65-pcb:SW_Cherry_MX_6.25u_PCB_Reversed_Stabilizer -> bakeneko:SW_Cherry_MX_6.25u_PCB_Reversed_Stabilizer
Changed lines of the file:
@@
 F 0 "MX65" H 10150 9085 50  0000 C CNN
 F 1 "6.25u" H 10150 8994 50  0000 C CNN
-F 2 "bakeneko-65-pcb:SW_Cherry_MX_6.25u_PCB_Reversed_Stabilizer" H 10150 8850 50  0001 C CNN
+F 2 "bakeneko:SW_Cherry_MX_6.25u_PCB_Reversed_Stabilizer" H 10150 8850 50  0001 C CNN
 F 3 "~" H 10150 8850 50  0001 C CNN
 	1    10150 8850

Commit message: Update
Changed lines of the file:
@@
-$EndComp
-$Comp
-L Switch:SW_SPST MX18
-U 1 1 5F2D2627
-P 6850 6750
-F 0 "MX18" H 6850 6985 50  0000 C CNN
-F 1 "1.5u" H 6850 6894 50  0000 C CNN
-F 2 "Button_Switch_Keyboard:SW_Cherry_MX_1.50u_PCB" H 6850 6750 50  0001 C CNN
-F 3 "~" H 6850 6750 50  0001 C CNN
-	1    6850 6750
-	1    0    0    1
 $EndComp
 $Comp
@@
 	6650 5450 6650 6050
 Connection ~ 6650 6050
-Wire Wire Line
-	6650 6050 6650 6750
-Connection ~ 6650 6750
-Wire Wire Line
-	6650 6750 6650 7450
 Connection ~ 6650 7450
 Wire Wire Line
@@
 	1    0    0    -1
 $EndComp
+$Comp
+L Switch:SW_SPST MX18
+U 1 1 5F325A2A
+P 6850 6750
+F 0 "MX18" H 6850 6985 50  0000 C CNN
+F 1 "1.5u" H 6850 6894 50  0000 C CNN
+F 2 "Button_Switch_Keyboard:SW_Cherry_MX_1.50u_PCB" H 6850 6750 50  0001 C CNN
+F 3 "~" H 6850 6750 50  0001 C CNN
+	1    6850 6750
+	1    0    0    -1
+$EndComp
+Wire Wire Line
+	6650 6050 6650 6750
+Connection ~ 6650 6750
+Wire Wire Line
+	6650 6750 6650 7450
 $EndSCHEMATC

Commit message: Add new stuff
Parts:
- removed D1, D10, D11, D12, D13, D14, D15, D16, D17, D18, D19, D2, D20, D21, D22, D23, D24, D25, D26, D27, D28, D29, D3, D30, D31, D32, D33, D34, D35, D36, D37, D38, D39, D4, D40, D41, D42, D43, D44, D45, D46, D47, D48, D49, D5, D50, D51, D52, D53, D54, D55, D56, D57, D58, D59, D6, D60, D61, D62, D63, D64, D65, D66, D67, D68, D69, D7, D8, D9: 1N4148, Diode_SMD:D_SOD-123, symbol Device:D
- removed MX1, MX10, MX11, MX12, MX13, MX14, MX15, MX16, MX19, MX2, MX20, MX21, MX22, MX23, MX24, MX25, MX26, MX27, MX28, MX29, MX3, MX30, MX32, MX35, MX36, MX37, MX38, MX39, MX4, MX40, MX41, MX42, MX43, MX44, MX45, MX47, MX49, MX5, MX50, MX51, MX52, MX53, MX54, MX55, MX56, MX57, MX58, MX6, MX60, MX61, MX66, MX67, MX68, MX69, MX7, MX70, MX71, MX8, MX9: 1u, Button_Switch_Keyboard:SW_Cherry_MX_1.00u_PCB, symbol Switch:SW_SPST
- removed MX17: 2u, Button_Switch_Keyboard:SW_Cherry_MX_2.00u_PCB, symbol Switch:SW_SPST
- removed MX18, MX31, MX72, MX73: 1.5u, Button_Switch_Keyboard:SW_Cherry_MX_1.50u_PCB, symbol Switch:SW_SPST
- removed MX33, MX62, MX63, MX64: 1.25u, Button_Switch_Keyboard:SW_Cherry_MX_1.25u_PCB, symbol Switch:SW_SPST
- removed MX34, MX59: 1.75u, Button_Switch_Keyboard:SW_Cherry_MX_1.75u_PCB, symbol Switch:SW_SPST
- removed MX46, MX48: 2.25u, Button_Switch_Keyboard:SW_Cherry_MX_2.25u_PCB, symbol Switch:SW_SPST
- removed MX65: 6.25u, bakeneko:SW_Cherry_MX_6.25u_PCB_Reversed_Stabilizer, symbol Switch:SW_SPST
Connections:
- net COL0: now also U2.37 (PF6); no longer U2.36 (PF7)
- net COL2: now also U2.40 (PF1); no longer U2.39 (PF4)
- net D+: now also U1.3 (IO2)
- net D-: now also U1.1 (IO1)
- net GND: now also U1.2 (GND)
- net ROW2: now also U2.36 (PF7); no longer U2.37 (PF6)
- net ROW3: now also U2.39 (PF4); no longer U2.38 (PF5)
- net ROW4: now also U2.38 (PF5); no longer U2.40 (PF1)
- net VBUS: now also U1.5 (VBUS)
- net ESD_D+: now reaches U1.4 (IO2)
- net ESD_D+: now also R2.2
- net ESD_D-: now reaches U1.6 (IO1)
- net ESD_D-: now also R3.2
- net MCU_D+: now reaches R2.1, U2.4 (D+)
- net MCU_D-: now reaches R3.1, U2.3 (D-)
- net VCC renamed +5V
Other:
- moved on the sheet: C1, C2, C3, C4, C5, C6, C7, F1, J1, J2, R1, R2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
