File: bakeneko-65-pcb.kicad_pcb (KiCad board)
At the start: 2 copper layers, 303.7 x 94.2 mm, 161 parts, among them J1 JST SH 4-pin, J2 AVR-ISP-6, SW1 Reset, U1 USBLC6-2SC6, U2 ATmega32U4-AU, Y1 16MHz

Commit message: Update PCB
Parts:
- moved F1 6.54 mm to (10.3, 13.5)
- moved U1 1.93 mm to (26.2, 14.6)
- moved J1 1.26 mm to (35.6, 14.6)
Connections:
- U1 pad 1: D+ -> D-
- U1 pad 3: D- -> D+
- U1 pad 4: Net-(R3-Pad2) -> Net-(R2-Pad2)
- U1 pad 6: Net-(R2-Pad2) -> Net-(R3-Pad2)
Routing:
- net VBUS: track 0.00 -> 9.87 mm
- net GND: track 0.00 -> 9.72 mm
- net D-: track 0.00 -> 6.45 mm
- net D+: track 0.00 -> 6.45 mm
Changed lines of the file:
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@@
     (thickness 1.6)
     (drawings 34)
-    (tracks 555)
+    (tracks 573)
     (zones 0)
     (modules 161)
@@
   )
   (module Package_TO_SOT_SMD:SOT-23-6 (layer B.Cu)
-    (at 27.78125 13.49375 180)
+    (at 26.19375 14.58375 180)
     (descr "6-pin SOT-23 package")
     (tags SOT-23-6)
@@
       (net 80 VBUS))
     (pad 6 smd rect (at 1.1 0.95 180) (size 1.06 0.65) (layers B.Cu B.Paste B.Mask)
-      (net 103 "Net-(R2-Pad2)"))
-    (pad 4 smd rect (at 1.1 -0.95 180) (size 1.06 0.65) (layers B.Cu B.Paste B.Mask)
       (net 105 "Net-(R3-Pad2)"))
+    (pad 4 smd rect (at 1.1 -0.95 180) (size 1.06 0.65) (layers B.Cu B.Paste B.Mask)
+      (net 103 "Net-(R2-Pad2)"))
     (pad 3 smd rect (at -1.1 -0.95 180) (size 1.06 0.65) (layers B.Cu B.Paste B.Mask)
-      (net 82 D-))
+      (net 81 D+))
     (pad 2 smd rect (at -1.1 0 180) (size 1.06 0.65) (layers B.Cu B.Paste B.Mask)
       (net 1 GND))
     (pad 1 smd rect (at -1.1 0.95 180) (size 1.06 0.65) (layers B.Cu B.Paste B.Mask)
-      (net 81 D+))
+      (net 82 D-))
     (model ${KISYS3DMOD}/Package_TO_SOT_SMD.3dshapes/SOT-23-6.wrl
       (at (xyz 0 0 0))
@@
   )
   (module Connector_JST:JST_SH_SM04B-SRSS-TB_1x04-1MP_P1.00mm_Horizontal (layer B.Cu)
-    (at 34.925 13.49375 270)
+    (at 35.56 14.58375 270)
     (descr "JST SH series connector, SM04B-SRSS-TB (http://www.jst-mfg.com/product/pdf/eng/eSH.pdf), generated with kicad-footprint-generator")
     (tags "connector JST SH top entry")
@@
   )
   (module Fuse:Fuse_1206_3216Metric (layer B.Cu)
-    (at 16.85625 13.49375)
+    (at 10.31875 13.49375)
     (descr "Fuse SMD 1206 (3216 Metric), square (rectangular) end terminal, IPC_7351 nominal, (Body size source: http://www.tortai-tech.com/upload/download/2011102023233369053.pdf), generated with kicad-footprint-generator")
     (tags resistor)
@@
   (gr_curve (pts (xy -10.954213 -3.334214) (xy -11.329286 -2.959141) (xy -11.54 -2.450433) (xy -11.54 -1.92)) (layer Edge.Cuts) (width 0.2))
   (gr_curve (pts (xy 292.209999 -1.92) (xy 292.209999 -3.024562) (xy 291.314581 -3.919989) (xy 290.210019 -3.92)) (layer Edge.Cuts) (width 0.2))
+  (segment (start 26.373249 14.896349) (end 26.685848 14.58375) (width 0.381) (layer B.Cu) (net 1))
+  (segment (start 26.373249 16.171151) (end 26.373249 14.896349) (width 0.381) (layer B.Cu) (net 1))
+  (segment (start 26.685848 14.58375) (end 27.29375 14.58375) (width 0.381) (layer B.Cu) (net 1))
+  (segment (start 26.585848 16.38375) (end 26.373249 16.171151) (width 0.381) (layer B.Cu) (net 1))
+  (segment (start 33.26 16.38375) (end 26.585848 16.38375) (width 0.381) (layer B.Cu) (net 1))
+  (segment (start 33.56 16.08375) (end 33.26 16.38375) (width 0.381) (layer B.Cu) (net 1))
   (segment (start 4.98375 2.54) (end 5.55625 3.1125) (width 0.25) (layer B.Cu) (net 6))
   (segment (start -6.35 2.54) (end 4.98375 2.54) (width 0.25) (layer B.Cu) (net 6))
@@
   (segment (start 276.00375 78.74) (end 275.43125 79.3125) (width 0.25) (layer B.Cu) (net 79))
   (segment (start 279.4 78.74) (end 276.00375 78.74) (width 0.25) (layer B.Cu) (net 79))
+  (segment (start 25.701652 14.58375) (end 25.09375 14.58375) (width 0.381) (layer B.Cu) (net 80))
+  (segment (start 26.19375 14.091652) (end 25.701652 14.58375) (width 0.381) (layer B.Cu) (net 80))
+  (segment (start 26.19375 13.175848) (end 26.19375 14.091652) (width 0.381) (layer B.Cu) (net 80))
+  (segment (start 26.585848 12.78375) (end 26.19375 13.175848) (width 0.381) (layer B.Cu) (net 80))
+  (segment (start 33.26 12.78375) (end 26.585848 12.78375) (width 0.381) (layer B.Cu) (net 80))
+  (segment (start 33.56 13.08375) (end 33.26 12.78375) (width 0.381) (layer B.Cu) (net 80))
+  (segment (start 32.335 15.53375) (end 27.29375 15.53375) (width 0.25) (layer B.Cu) (net 81))
+  (segment (start 32.785 15.08375) (end 32.335 15.53375) (width 0.25) (layer B.Cu) (net 81))
+  (segment (start 33.56 15.08375) (end 32.785 15.08375) (width 0.25) (layer B.Cu) (net 81))
+  (segment (start 32.335 13.63375) (end 27.29375 13.63375) (width 0.25) (layer B.Cu) (net 82))
+  (segment (start 32.785 14.08375) (end 32.335 13.63375) (width 0.25) (layer B.Cu) (net 82))
+  (segment (start 33.56 14.08375) (end 32.785 14.08375) (width 0.25) (layer B.Cu) (net 82))
   (segment (start 0 14.2875) (end 4.7625 19.05) (width 0.25) (layer F.Cu) (net 87))
   (segment (start 0 0) (end 0 14.2875) (width 0.25) (layer F.Cu) (net 87))

Commit message: Update bakeneko-65-pcb.kicad_pcb
Parts:
- moved F1 10.3 mm to (20.1, 10.3)
- moved R2 4.33 mm to (20.1, 16.0)
- moved R3 2.34 mm to (20.1, 13.1)
Routing:
- net COL4: track 125.7 -> 67.0 mm
- net VBUS: track 9.87 -> 17.0 mm, vias 0 -> 2
- net Net-(R3-Pad2): track 0.00 -> 4.52 mm
- net Net-(R2-Pad2): track 0.00 -> 4.23 mm
Changed lines of the file:
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@@
     (thickness 1.6)
     (drawings 34)
-    (tracks 573)
+    (tracks 587)
     (zones 0)
     (modules 161)
@@
   )
   (module Resistor_SMD:R_0805_2012Metric (layer B.Cu)
-    (at 21.43125 15.08125)
+    (at 20.13125 13.13375)
     (descr "Resistor SMD 0805 (2012 Metric), square (rectangular) end terminal, IPC_7351 nominal, (Body size source: https://docs.google.com/spreadsheets/d/1BsfQQcO9C6DZCsRaXUlFlo91Tg2WpOkGARC1WS5S8t0/edit?usp=sharing), generated with kicad-footprint-generator")
     (tags resistor)
@@
   )
   (module Resistor_SMD:R_0805_2012Metric (layer B.Cu)
-    (at 21.43125 11.90625)
+    (at 20.13125 16.03375)
     (descr "Resistor SMD 0805 (2012 Metric), square (rectangular) end terminal, IPC_7351 nominal, (Body size source: https://docs.google.com/spreadsheets/d/1BsfQQcO9C6DZCsRaXUlFlo91Tg2WpOkGARC1WS5S8t0/edit?usp=sharing), generated with kicad-footprint-generator")
     (tags resistor)
@@
   )
   (module Fuse:Fuse_1206_3216Metric (layer B.Cu)
-    (at 10.31875 13.49375)
+    (at 20.13125 10.31875)
     (descr "Fuse SMD 1206 (3216 Metric), square (rectangular) end terminal, IPC_7351 nominal, (Body size source: http://www.tortai-tech.com/upload/download/2011102023233369053.pdf), generated with kicad-footprint-generator")
     (tags resistor)
@@
       (effects (font (size 1 1) (thickness 0.15)) (justify mirror))
     )
-    (fp_text user %R (at 0 0) (layer B.Fab)
+    (fp_text user %R (at -4.3 0) (layer B.Fab)
       (effects (font (size 0.8 0.8) (thickness 0.12)) (justify mirror))
     )
@@
   (segment (start 33.26 12.78375) (end 26.585848 12.78375) (width 0.381) (layer B.Cu) (net 80))
   (segment (start 33.56 13.08375) (end 33.26 12.78375) (width 0.381) (layer B.Cu) (net 80))
+  (via (at 23.8125 14.2875) (size 0.8) (drill 0.4) (layers F.Cu B.Cu) (net 80))
+  (segment (start 25.09375 14.58375) (end 24.10875 14.58375) (width 0.381) (layer B.Cu) (net 80))
+  (segment (start 24.10875 14.58375) (end 23.8125 14.2875) (width 0.381) (layer B.Cu) (net 80))
+  (via (at 23.8125 11.90625) (size 0.8) (drill 0.4) (layers F.Cu B.Cu) (net 80))
+  (segment (start 23.8125 14.2875) (end 23.8125 11.90625) (width 0.381) (layer F.Cu) (net 80))
+  (segment (start 23.8125 11.3) (end 22.83125 10.31875) (width 0.381) (layer B.Cu) (net 80))
+  (segment (start 23.8125 11.90625) (end 23.8125 11.3) (width 0.381) (layer B.Cu) (net 80))
+  (segment (start 22.83125 10.31875) (end 21.53125 10.31875) (width 0.381) (layer B.Cu) (net 80))
   (segment (start 32.335 15.53375) (end 27.29375 15.53375) (width 0.25) (layer B.Cu) (net 81))
   (segment (start 32.785 15.08375) (end 32.335 15.53375) (width 0.25) (layer B.Cu) (net 81))
@@
   (segment (start 11.90625 66.675) (end 2.38125 76.2) (width 0.25) (layer F.Cu) (net 87))
   (segment (start 11.90625 57.15) (end 11.90625 66.675) (width 0.25) (layer F.Cu) (net 87))
-  (segment (start 19.05 9.525) (end 28.575 19.05) (width 0.25) (layer F.Cu) (net 88))
-  (segment (start 19.05 0) (end 19.05 9.525) (width 0.25) (layer F.Cu) (net 88))
   (segment (start 28.575 33.3375) (end 33.3375 38.1) (width 0.25) (layer F.Cu) (net 88))
   (segment (start 28.575 19.05) (end 28.575 33.3375) (width 0.25) (layer F.Cu) (net 88))
   (segment (start 33.3375 69.05625) (end 26.19375 76.2) (width 0.25) (layer F.Cu) (net 88))
   (segment (start 33.3375 38.1) (end 33.3375 69.05625) (width 0.25) (layer F.Cu) (net 88))
+  (segment (start 28.575 9.525) (end 28.575 19.05) (width 0.25) (layer F.Cu) (net 88))
+  (segment (start 19.05 0) (end 28.575 9.525) (width 0.25) (layer F.Cu) (net 88))
   (segment (start 38.1 9.525) (end 47.625 19.05) (width 0.25) (layer F.Cu) (net 89))
   (segment (start 38.1 0) (end 38.1 9.525) (width 0.25) (layer F.Cu) (net 89))
@@
   (segment (start 90.4875 47.625) (end 80.9625 57.15) (width 0.25) (layer F.Cu) (net 91))
   (segment (start 90.4875 38.1) (end 90.4875 47.625) (width 0.25) (layer F.Cu) (net 91))
-  (segment (start 89.062499 36.674999) (end 32.381251 36.674999) (width 0.25) (layer B.Cu) (net 91))
-  (segment (start 90.4875 38.1) (end 89.062499 36.674999) (width 0.25) (layer B.Cu) (net 91))
   (segment (start 95.25 9.525) (end 104.775 19.05) (width 0.25) (layer F.Cu) (net 92))
   (segment (start 95.25 0) (end 95.25 9.525) (width 0.25) (layer F.Cu) (net 92))
@@
   (segment (start 285.75 19.05) (end 285.75 38.1) (width 0.25) (layer F.Cu) (net 102))
   (segment (start 285.75 38.1) (end 285.75 76.2) (width 0.25) (layer F.Cu) (net 102))
+  (segment (start 24.55875 16.03375) (end 22.36875 16.03375) (width 0.25) (layer B.Cu) (net 103))
+  (segment (start 25.05875 15.53375) (end 24.55875 16.03375) (width 0.25) (layer B.Cu) (net 103))
+  (segment (start 25.09375 15.53375) (end 25.05875 15.53375) (width 0.25) (layer B.Cu) (net 103))
+  (segment (start 22.36875 16.03375) (end 21.06875 16.03375) (width 0.25) (layer B.Cu) (net 103))
+  (segment (start 24.59375 13.13375) (end 25.09375 13.63375) (width 0.25) (layer B.Cu) (net 105))
+  (segment (start 21.06875 13.13375) (end 22.65875 13.13375) (width 0.25) (layer B.Cu) (net 105))
+  (segment (start 22.36875 13.13375) (end 22.65875 13.13375) (width 0.25) (layer B.Cu) (net 105))
+  (segment (start 22.65875 13.13375) (end 24.59375 13.13375) (width 0.25) (layer B.Cu) (net 105))
 )

Commit message: Update bakeneko-65-pcb.kicad_pcb
Parts:
- removed C8: 1u, Capacitor_SMD:C_0805_2012Metric
- C4: value 0.1u -> 10u
- C5: value 4.7u -> 22p
- C7: value 22p -> 1u
- moved C7 53.1 mm to (-34.5, 30.5), turned to 180 degrees
- moved C4 49.2 mm to (-33.2, 36.0)
- moved C2 45.5 mm to (-18.5, 40.8)
- moved U2 41.3 mm to (-23.6, 30.6)
- moved C1 40.8 mm to (-32.2, 21.9), turned to 270 degrees
- moved C3 39.9 mm to (-14.8, 25.3)
- moved R4 39.6 mm to (-14.9, 34.0)
- moved Y1 38.9 mm to (-24.0, 19.2)
- moved SW1 38.9 mm to (7.18, 11.9)
- moved C5 38.5 mm to (-28.0, 19.2), turned to 90 degrees
- moved R1 31.7 mm to (7.67, 16.2)
- moved C6 30.7 mm to (-19.9, 19.2), turned to 270 degrees
- moved U1 1.19 mm to (27.4, 14.6)
- moved J2 0.83 mm to (-3.97, 32.0)
- moved R2 0.70 mm to (20.8, 15.8)
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Connections:
- C5 pad 1: VCC -> GND
- C5 pad 2: GND -> XTAL2
- C6 pad 2: XTAL2 -> XTAL1
- C7 pad 1: GND -> Net-(C7-Pad1)
- C7 pad 2: XTAL1 -> GND
- U2 pad 1: Net-(U2-Pad1) -> ROW2
- U2 pad 12: ROW4 -> Net-(U2-Pad12)
- U2 pad 18: Net-(U2-Pad18) -> ROW1
- U2 pad 40: Net-(U2-Pad40) -> ROW3
- U2 pad 41: Net-(U2-Pad41) -> ROW4
- U2 pad 6: Net-(C8-Pad1) -> Net-(C7-Pad1)
Routing:
- net ROW3: track 284.6 -> 0.00 mm
- net ROW0: track 280.7 -> 0.00 mm
- net ROW4: track 272.7 -> 0.00 mm
- net ROW1: track 251.3 -> 0.00 mm
- net ROW2: track 245.6 -> 0.00 mm
- net COL9: track 96.7 -> 0.00 mm
- net COL11: track 94.8 -> 0.00 mm
- net COL10: track 92.0 -> 0.00 mm
- net COL13: track 91.0 -> 0.00 mm
- net COL0: track 89.8 -> 0.00 mm
- net COL2: track 89.0 -> 0.00 mm
- net COL6: track 87.0 -> 0.00 mm
- net COL1: track 85.1 -> 0.00 mm
- net COL12: track 84.2 -> 0.00 mm
- net COL15: track 76.2 -> 0.00 mm
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
Commit message: Update bakeneko-65-pcb.kicad_pcb
Parts:
- moved C1 57.9 mm to (25.6, 25.2), turned to 180 degrees
- moved C5 57.4 mm to (28.4, 29.4), turned to 0 degrees
- moved Y1 54.3 mm to (28.4, 33.4), turned to 90 degrees
- moved C6 51.7 mm to (28.4, 37.5), turned to 180 degrees
- moved C7 46.8 mm to (11.8, 23.4), turned to 90 degrees
- moved C4 46.5 mm to (11.3, 22.5)
- moved C3 40.9 mm to (22.3, 42.7), turned to 180 degrees
- moved U2 40.7 mm to (17.0, 33.8), turned to 270 degrees
- moved R1 32.2 mm to (-24.5, 17.1)
- moved SW1 31.2 mm to (-24.0, 10.1)
- moved R4 29.7 mm to (13.5, 42.5), turned to 0 degrees
- moved C2 25.3 mm to (6.78, 39.0), turned to 90 degrees
- moved F1 7.60 mm to (13.8, 14.6)
Routing:
- net VBUS: track 0.00 -> 22.7 mm, vias 0 -> 2
- net Net-(R3-Pad1): track 0.00 -> 17.3 mm
- net Net-(R2-Pad1): track 0.00 -> 15.5 mm
- net GND: track 21.9 -> 8.56 mm
- net XTAL2: track 10.2 -> 0.00 mm
- net XTAL1: track 8.13 -> 0.00 mm
- net VCC: track 0.00 -> 7.42 mm
- net D-: track 0.00 -> 5.27 mm
- net D+: track 0.00 -> 5.27 mm
- net Net-(R2-Pad2): track 0.00 -> 4.67 mm
- net Net-(R3-Pad2): track 0.00 -> 4.67 mm

Commit message: Update bakeneko-65-pcb.kicad_pcb
Parts:
- moved SW1 71.0 mm to (43.7, 31.6)
- moved R1 60.8 mm to (34.8, 30.5), turned to 180 degrees
- moved C7 6.03 mm to (17.7, 22.5)
- moved C2 4.47 mm to (5.63, 34.6), turned to 0 degrees
- moved C1 4.02 mm to (28.4, 28.1)
- moved C3 2.81 mm to (20.3, 44.7), turned to 270 degrees
- moved R4 2.35 mm to (12.7, 44.7), turned to 90 degrees
- moved C5 1.10 mm to (28.4, 30.5)
- moved Y1 0.60 mm to (28.4, 34.0)
- moved C6 0.10 mm to (28.4, 37.6)
Routing:
- net GND: track 8.56 -> 140.1 mm
- net VCC: track 7.42 -> 102.2 mm, vias 0 -> 6
- net RESET: track 0.00 -> 28.9 mm
- net XTAL2: track 0.00 -> 10.0 mm
- net XTAL1: track 0.00 -> 7.87 mm
- net Net-(C7-Pad1): track 0.00 -> 5.03 mm
- net Net-(R4-Pad2): track 0.00 -> 4.32 mm

Commit message: Update PCB
Parts:
- moved J2 17.7 mm to (-5.08, 14.3), turned to 0 degrees
- moved C6 5.53 mm to (32.8, 34.2)
- moved C5 4.58 mm to (32.8, 31.9), turned to 180 degrees
- moved R1 2.44 mm to (32.8, 29.1)
- moved C1 1.00 mm to (28.4, 29.1), turned to 0 degrees
- moved Y1 1.00 mm to (28.4, 33.0)
Connections:
- U2 pad 1: ROW2 -> ROW0
- U2 pad 12: Net-(U2-Pad12) -> ROW1
- U2 pad 18: ROW1 -> Net-(U2-Pad18)
- U2 pad 19: COL15 -> Net-(U2-Pad19)
- U2 pad 20: COL14 -> Net-(U2-Pad20)
- U2 pad 21: COL13 -> Net-(U2-Pad21)
- U2 pad 22: COL12 -> Net-(U2-Pad22)
- U2 pad 25: COL11 -> Net-(U2-Pad25)
- U2 pad 26: COL10 -> Net-(U2-Pad26)
- U2 pad 27: COL9 -> Net-(U2-Pad27)
- U2 pad 28: COL8 -> Net-(U2-Pad28)
- U2 pad 29: COL7 -> Net-(U2-Pad29)
- U2 pad 30: COL6 -> Net-(U2-Pad30)
- U2 pad 31: COL5 -> Net-(U2-Pad31)
- U2 pad 32: COL4 -> Net-(U2-Pad32)
- U2 pad 36: COL1 -> Net-(U2-Pad36)
- U2 pad 37: COL3 -> Net-(U2-Pad37)
- U2 pad 38: COL2 -> Net-(U2-Pad38)
- U2 pad 39: COL0 -> Net-(U2-Pad39)
- U2 pad 40: ROW3 -> Net-(U2-Pad40)
- U2 pad 41: ROW4 -> COL0
- U2 pad 8: ROW0 -> COL1
Routing:
- net COL1: track 0.00 -> 106.2 mm
- net COL11: track 0.00 -> 96.9 mm
- net COL9: track 0.00 -> 96.7 mm
- net COL10: track 0.00 -> 92.0 mm
- net COL13: track 0.00 -> 90.1 mm
- net COL0: track 0.00 -> 89.8 mm
- net COL2: track 0.00 -> 89.0 mm
- net COL6: track 0.00 -> 87.0 mm
- net COL12: track 0.00 -> 84.2 mm
- net COL15: track 0.00 -> 76.2 mm
- net MISO: track 0.00 -> 74.1 mm
- net SCK: track 0.00 -> 71.4 mm
- net RESET: track 28.9 -> 96.6 mm, vias 0 -> 2
- net COL8: track 0.00 -> 67.0 mm
- net COL3: track 0.00 -> 67.0 mm
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
Commit message: Update PCB
Parts:
- moved D32 15.2 mm to (9.65, 47.6)
- moved D60 1.74 mm to (9.65, 81.3)
- moved D33 0.74 mm to (38.2, 43.2)
- moved D1 0.74 mm to (4.88, 5.08)
- moved D18 0.74 mm to (33.5, 24.1)
- moved D14 0.74 mm to (233.5, 5.08)
- moved D66 0.74 mm to (233.5, 81.3)
- moved D53 0.52 mm to (147.2, 62.2)
- moved C1 0.50 mm to (28.4, 28.6)
- moved R1 0.50 mm to (32.8, 28.6)
- moved D45 0.48 mm to (275.8, 43.2)
- moved D16 0.48 mm to (275.8, 5.08)
- moved D31 0.48 mm to (275.8, 24.1)
- moved D59 0.48 mm to (275.8, 62.2)
- moved D69 0.48 mm to (275.8, 81.3)
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Connections:
- U2 pad 18: Net-(U2-Pad18) -> COL15
- U2 pad 19: Net-(U2-Pad19) -> COL14
- U2 pad 20: Net-(U2-Pad20) -> COL13
- U2 pad 21: Net-(U2-Pad21) -> COL12
- U2 pad 22: Net-(U2-Pad22) -> COL11
- U2 pad 25: Net-(U2-Pad25) -> COL10
- U2 pad 26: Net-(U2-Pad26) -> COL9
- U2 pad 27: Net-(U2-Pad27) -> COL8
- U2 pad 28: Net-(U2-Pad28) -> COL7
- U2 pad 29: Net-(U2-Pad29) -> COL6
- U2 pad 30: Net-(U2-Pad30) -> COL5
- U2 pad 31: Net-(U2-Pad31) -> COL4
- U2 pad 32: Net-(U2-Pad32) -> COL3
- U2 pad 36: Net-(U2-Pad36) -> COL0
- U2 pad 37: Net-(U2-Pad37) -> ROW2
- U2 pad 38: Net-(U2-Pad38) -> ROW3
- U2 pad 39: Net-(U2-Pad39) -> COL2
- U2 pad 40: Net-(U2-Pad40) -> ROW4
- U2 pad 41: COL0 -> Net-(U2-Pad41)
Routing:
- net ROW4: track 0.00 -> 360.1 mm, vias 0 -> 2
- net ROW3: track 0.00 -> 340.1 mm, vias 0 -> 2
- net ROW2: track 0.00 -> 325.9 mm, vias 0 -> 4
- net ROW0: track 2.17 -> 326.0 mm, vias 1 -> 2
- net COL14: track 9.52 -> 321.4 mm, vias 0 -> 1
- net COL15: track 76.2 -> 360.3 mm
- net ROW1: track 13.2 -> 293.1 mm, vias 0 -> 2
- net COL13: track 90.1 -> 354.1 mm
- net COL12: track 84.2 -> 323.5 mm
- net COL11: track 96.9 -> 306.5 mm
- net COL10: track 92.0 -> 282.5 mm
- net COL9: track 96.7 -> 268.7 mm
- net COL8: track 67.0 -> 220.7 mm
- net COL7: track 67.0 -> 202.3 mm
- net COL2: track 89.0 -> 215.9 mm, vias 0 -> 2
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- added copper zone on B.Cu, net GND

Commit message: Update bakeneko-65-pcb.kicad_pcb
Other:
- board text added: "Bakeneko 65 v1.0"
