File: bakeneko-65-pcb.kicad_pcb (KiCad board)
At the start: 2 copper layers, 303.8 x 94.2 mm, 160 parts, among them J1 JST SH 4-pin, J2 AVR-ISP-6, SW1 Reset, U1 USBLC6-2SC6, U2 ATmega32U4-AU, Y1 16MHz

Commit message: Update bakeneko-65-pcb.kicad_pcb
Parts:
- moved F1 1.00 mm to (13.8, 13.6)
- moved J1 1.00 mm to (35.6, 13.6)
- moved R2 1.00 mm to (20.8, 14.8)
- moved R3 1.00 mm to (20.8, 12.3)
- moved U1 1.00 mm to (27.4, 13.6)
Routing:
- net SCK: track 72.7 -> 36.1 mm, vias 0 -> 2
- net MOSI: track 71.0 -> 34.6 mm, vias 0 -> 2
- net MISO: track 74.9 -> 44.5 mm
- net RESET: track 97.0 -> 99.5 mm
- net Net-(R2-Pad1): track 15.1 -> 16.9 mm
- net GND: track 162.7 -> 160.9 mm
- net Net-(R3-Pad1): track 17.3 -> 18.6 mm
- net VCC: track 106.5 -> 107.8 mm
- net COL1: track 106.2 -> 107.5 mm, vias 0 -> 1

Commit message: Update bakeneko-65-pcb.kicad_pcb
Routing:
- net GND: track 160.9 -> 184.8 mm, vias 4 -> 8
Changed lines of the file:
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@@
     (thickness 1.6)
     (drawings 53)
-    (tracks 1023)
+    (tracks 1039)
     (zones 0)
     (modules 160)
@@
   (segment (start 30.5125 29.75) (end 31.5725 29.75) (width 0.381) (layer B.Cu) (net 1))
   (segment (start 40.55375 33.465) (end 40.415 33.465) (width 0.381) (layer B.Cu) (net 1))
-  (segment (start 36.7 29.75) (end 31.5725 29.75) (width 0.381) (layer B.Cu) (net 1))
-  (segment (start 40.415 33.465) (end 36.7 29.75) (width 0.381) (layer B.Cu) (net 1))
   (segment (start 16.21375 18.03625) (end 16.21375 19.03625) (width 0.381) (layer B.Cu) (net 1))
   (segment (start 0.882499 11.807501) (end 0.96 11.73) (width 0.381) (layer B.Cu) (net 1))
@@
   (segment (start 9.65 20.47) (end 9.65 21.4) (width 0.381) (layer F.Cu) (net 1))
   (segment (start 0.96 11.78) (end 9.65 20.47) (width 0.381) (layer F.Cu) (net 1))
+  (via (at 21.674956 47.33) (size 0.8) (drill 0.4) (layers F.Cu B.Cu) (net 1))
+  (segment (start 20.313749 45.60625) (end 20.313749 45.968793) (width 0.381) (layer B.Cu) (net 1))
+  (segment (start 20.313749 45.968793) (end 21.674956 47.33) (width 0.381) (layer B.Cu) (net 1))
+  (via (at 25.06 47.33) (size 0.8) (drill 0.4) (layers F.Cu B.Cu) (net 1))
+  (segment (start 21.674956 47.33) (end 25.06 47.33) (width 0.381) (layer F.Cu) (net 1))
+  (segment (start 39.46 34.63) (end 40.55375 33.53625) (width 0.381) (layer B.Cu) (net 1))
+  (segment (start 26.16 48.43) (end 32.869598 48.43) (width 0.381) (layer B.Cu) (net 1))
+  (segment (start 25.06 47.33) (end 26.16 48.43) (width 0.381) (layer B.Cu) (net 1))
+  (segment (start 40.55375 33.53625) (end 40.55375 33.465) (width 0.381) (layer B.Cu) (net 1))
+  (via (at 34.092711 47.934484) (size 0.8) (drill 0.4) (layers F.Cu B.Cu) (net 1))
+  (segment (start 32.869598 48.43) (end 33.597195 48.43) (width 0.381) (layer B.Cu) (net 1))
+  (segment (start 33.597195 48.43) (end 34.092711 47.934484) (width 0.381) (layer B.Cu) (net 1))
+  (via (at 35.71 38.33) (size 0.8) (drill 0.4) (layers F.Cu B.Cu) (net 1))
+  (segment (start 34.092711 47.934484) (end 34.092711 39.947289) (width 0.381) (layer F.Cu) (net 1))
+  (segment (start 34.092711 39.947289) (end 35.71 38.33) (width 0.381) (layer F.Cu) (net 1))
+  (segment (start 35.71 38.33) (end 38.66 38.33) (width 0.381) (layer B.Cu) (net 1))
+  (segment (start 39.46 37.53) (end 39.46 34.63) (width 0.381) (layer B.Cu) (net 1))
+  (segment (start 38.66 38.33) (end 39.46 37.53) (width 0.381) (layer B.Cu) (net 1))
   (segment (start 13.81375 26.38625) (end 13.81375 28.13875) (width 0.381) (layer B.Cu) (net 2))
   (via (at 13.81375 26.38625) (size 0.8) (drill 0.4) (layers F.Cu B.Cu) (net 2))

Commit message: Update bakeneko-65-pcb.kicad_pcb
Routing:
- net GND: track 184.8 -> 187.2 mm
