File: bakeneko-65-pcb.kicad_pcb (KiCad board)
At the start: 2 copper layers, 303.8 x 94.2 mm, 160 parts, among them J1 JST SH 4-pin, J2 AVR-ISP-6, SW1 Reset, U1 USBLC6-2SC6, U2 ATmega32U4-AU, Y1 16MHz

Commit message: Add new stuff
Parts:
- MX1, MX10, MX11, MX12, MX13, MX14, MX15, MX16, MX19, MX2, MX20, MX21, MX22, MX23, MX24, MX25, MX26, MX27, MX28, MX29, MX3, MX30, MX32, MX35, MX36, MX37, MX38, MX39, MX4, MX40, MX41, MX42, MX43, MX44, MX45, MX47, MX49, MX5, MX50, MX51, MX52, MX53, MX54, MX55, MX56, MX57, MX58, MX6, MX60, MX61, MX66, MX67, MX68, MX69, MX7, MX70, MX71, MX8, MX9: footprint Button_Switch_Keyboard:SW_Cherry_MX_1.00u_PCB -> MX_Only:MXOnly-1U-NoLED
- MX17: footprint Button_Switch_Keyboard:SW_Cherry_MX_2.00u_PCB -> MX_Only:MXOnly-2U-NoLED
- MX18, MX31, MX72, MX73: footprint Button_Switch_Keyboard:SW_Cherry_MX_1.50u_PCB -> MX_Only:MXOnly-1.5U-NoLED
- MX33, MX62, MX63, MX64: footprint Button_Switch_Keyboard:SW_Cherry_MX_1.25u_PCB -> MX_Only:MXOnly-1.25U-NoLED
- MX34, MX59: footprint Button_Switch_Keyboard:SW_Cherry_MX_1.75u_PCB -> MX_Only:MXOnly-1.75U-NoLED
- MX46, MX48: footprint Button_Switch_Keyboard:SW_Cherry_MX_2.25u_PCB -> MX_Only:MXOnly-2.25U-NoLED
- MX65: footprint bakeneko:SW_Cherry_MX_6.25u_PCB_Reversed_Stabilizer -> MX_Only:MXOnly-6.25U-ReversedStabilizers-NoLED
- moved D16 22.8 mm to (253.0, 5.87)
- moved D18 22.8 mm to (56.2, 24.9)
- moved D15 18.7 mm to (256.4, 5.87)
- moved MX17 17.3 mm to (273.7, 5.08)
- moved D19 15.4 mm to (53.0, 24.9)
- moved D20 15.4 mm to (72.1, 24.9)
- moved D46 15.4 mm to (17.3, 63.0)
- moved R4 9.23 mm to (18.3, 52.0)
- moved R1 5.76 mm to (38.2, 30.6), turned to 270 degrees
- moved MX12 5.68 mm to (207.0, 5.08)
- moved MX16 5.68 mm to (283.2, 5.08)
- moved MX26 5.68 mm to (159.4, 24.1)
- moved MX31 5.68 mm to (259.4, 24.1)
- moved MX32 5.68 mm to (283.2, 24.1)
- moved MX43 5.68 mm to (183.2, 43.2)
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Connections:
- net Net-(R2-Pad1) renamed /MCU_D+
- net Net-(R2-Pad2) renamed ESD_D+
- net Net-(R3-Pad1) renamed /MCU_D-
- net Net-(R3-Pad2) renamed ESD_D-
- net VCC renamed +5V
- MX1 pad 1: COL0 -> Net-(D1-Pad2)
- MX1 pad 2: Net-(D1-Pad2) -> COL0
- MX10 pad 1: COL9 -> Net-(D10-Pad2)
- MX10 pad 2: Net-(D10-Pad2) -> COL9
- MX11 pad 1: COL10 -> Net-(D11-Pad2)
- MX11 pad 2: Net-(D11-Pad2) -> COL10
- MX12 pad 1: COL11 -> Net-(D12-Pad2)
- MX12 pad 2: Net-(D12-Pad2) -> COL11
- MX13 pad 1: COL12 -> Net-(D13-Pad2)
- MX13 pad 2: Net-(D13-Pad2) -> COL12
- MX14 pad 1: COL13 -> Net-(D14-Pad2)
- MX14 pad 2: Net-(D14-Pad2) -> COL13
- MX15 pad 1: COL14 -> Net-(D15-Pad2)
- MX15 pad 2: Net-(D15-Pad2) -> COL14
- MX16 pad 1: COL15 -> Net-(D16-Pad2)
- MX16 pad 2: Net-(D16-Pad2) -> COL15
- MX17 pad 1: COL14 -> Net-(D15-Pad2)
- MX17 pad 2: Net-(D15-Pad2) -> COL14
- MX18 pad 1: COL0 -> Net-(D17-Pad2)
- MX18 pad 2: Net-(D17-Pad2) -> COL0
- MX19 pad 1: COL1 -> Net-(D18-Pad2)
- MX19 pad 2: Net-(D18-Pad2) -> COL1
- MX2 pad 1: COL1 -> Net-(D2-Pad2)
- MX2 pad 2: Net-(D2-Pad2) -> COL1
- MX20 pad 1: COL2 -> Net-(D19-Pad2)
- MX20 pad 2: Net-(D19-Pad2) -> COL2
- MX21 pad 1: COL3 -> Net-(D20-Pad2)
- MX21 pad 2: Net-(D20-Pad2) -> COL3
- MX22 pad 1: COL4 -> Net-(D21-Pad2)
- MX22 pad 2: Net-(D21-Pad2) -> COL4
- MX23 pad 1: COL5 -> Net-(D22-Pad2)
- MX23 pad 2: Net-(D22-Pad2) -> COL5
- MX24 pad 1: COL6 -> Net-(D23-Pad2)
- MX24 pad 2: Net-(D23-Pad2) -> COL6
- MX25 pad 1: COL7 -> Net-(D24-Pad2)
- MX25 pad 2: Net-(D24-Pad2) -> COL7
- MX26 pad 1: COL8 -> Net-(D25-Pad2)
- MX26 pad 2: Net-(D25-Pad2) -> COL8
- MX27 pad 1: COL9 -> Net-(D26-Pad2)
- MX27 pad 2: Net-(D26-Pad2) -> COL9
- MX28 pad 1: COL10 -> Net-(D27-Pad2)
- MX28 pad 2: Net-(D27-Pad2) -> COL10
- MX29 pad 1: COL11 -> Net-(D28-Pad2)
- MX29 pad 2: Net-(D28-Pad2) -> COL11
- MX3 pad 1: COL2 -> Net-(D3-Pad2)
- MX3 pad 2: Net-(D3-Pad2) -> COL2
- MX30 pad 1: COL12 -> Net-(D29-Pad2)
- MX30 pad 2: Net-(D29-Pad2) -> COL12
- MX31 pad 1: COL13 -> Net-(D30-Pad2)
- MX31 pad 2: Net-(D30-Pad2) -> COL13
- MX32 pad 1: COL15 -> Net-(D31-Pad2)
- MX32 pad 2: Net-(D31-Pad2) -> COL15
- MX33 pad 1: COL0 -> Net-(D32-Pad2)
- MX33 pad 2: Net-(D32-Pad2) -> COL0
- MX34 pad 1: COL0 -> Net-(D32-Pad2)
- MX34 pad 2: Net-(D32-Pad2) -> COL0
- MX35 pad 1: COL1 -> Net-(D33-Pad2)
- MX35 pad 2: Net-(D33-Pad2) -> COL1
- MX36 pad 1: COL2 -> Net-(D34-Pad2)
- MX36 pad 2: Net-(D34-Pad2) -> COL2
- MX37 pad 1: COL3 -> Net-(D35-Pad2)
- MX37 pad 2: Net-(D35-Pad2) -> COL3
- MX38 pad 1: COL4 -> Net-(D36-Pad2)
- MX38 pad 2: Net-(D36-Pad2) -> COL4
- MX39 pad 1: COL5 -> Net-(D37-Pad2)
- MX39 pad 2: Net-(D37-Pad2) -> COL5
- MX4 pad 1: COL3 -> Net-(D4-Pad2)
- MX4 pad 2: Net-(D4-Pad2) -> COL3
- MX40 pad 1: COL6 -> Net-(D38-Pad2)
- MX40 pad 2: Net-(D38-Pad2) -> COL6
- MX41 pad 1: COL7 -> Net-(D39-Pad2)
- MX41 pad 2: Net-(D39-Pad2) -> COL7
- MX42 pad 1: COL8 -> Net-(D40-Pad2)
- MX42 pad 2: Net-(D40-Pad2) -> COL8
- MX43 pad 1: COL9 -> Net-(D41-Pad2)
- MX43 pad 2: Net-(D41-Pad2) -> COL9
- MX44 pad 1: COL10 -> Net-(D42-Pad2)
- MX44 pad 2: Net-(D42-Pad2) -> COL10
- MX45 pad 1: COL11 -> Net-(D43-Pad2)
- MX45 pad 2: Net-(D43-Pad2) -> COL11
- MX46 pad 1: COL13 -> Net-(D44-Pad2)
- MX46 pad 2: Net-(D44-Pad2) -> COL13
- MX47 pad 1: COL15 -> Net-(D45-Pad2)
- MX47 pad 2: Net-(D45-Pad2) -> COL15
- MX48 pad 1: COL0 -> Net-(D46-Pad2)
- MX48 pad 2: Net-(D46-Pad2) -> COL0
- MX49 pad 1: COL2 -> Net-(D47-Pad2)
- MX49 pad 2: Net-(D47-Pad2) -> COL2
- MX5 pad 1: COL4 -> Net-(D5-Pad2)
- MX5 pad 2: Net-(D5-Pad2) -> COL4
- MX50 pad 1: COL3 -> Net-(D48-Pad2)
- MX50 pad 2: Net-(D48-Pad2) -> COL3
- MX51 pad 1: COL4 -> Net-(D49-Pad2)
- MX51 pad 2: Net-(D49-Pad2) -> COL4
- MX52 pad 1: COL5 -> Net-(D50-Pad2)
- MX52 pad 2: Net-(D50-Pad2) -> COL5
- MX53 pad 1: COL6 -> Net-(D51-Pad2)
- MX53 pad 2: Net-(D51-Pad2) -> COL6
- MX54 pad 1: COL7 -> Net-(D52-Pad2)
- MX54 pad 2: Net-(D52-Pad2) -> COL7
- MX55 pad 1: COL8 -> Net-(D53-Pad2)
- MX55 pad 2: Net-(D53-Pad2) -> COL8
- MX56 pad 1: COL9 -> Net-(D54-Pad2)
- MX56 pad 2: Net-(D54-Pad2) -> COL9
- MX57 pad 1: COL10 -> Net-(D55-Pad2)
- MX57 pad 2: Net-(D55-Pad2) -> COL10
- MX58 pad 1: COL11 -> Net-(D56-Pad2)
- MX58 pad 2: Net-(D56-Pad2) -> COL11
- MX59 pad 1: COL12 -> Net-(D57-Pad2)
- MX59 pad 2: Net-(D57-Pad2) -> COL12
- MX6 pad 1: COL5 -> Net-(D6-Pad2)
- MX6 pad 2: Net-(D6-Pad2) -> COL5
- MX60 pad 1: COL13 -> Net-(D58-Pad2)
- MX60 pad 2: Net-(D58-Pad2) -> COL13
- MX61 pad 1: COL15 -> Net-(D59-Pad2)
- MX61 pad 2: Net-(D59-Pad2) -> COL15
- MX62 pad 1: COL0 -> Net-(D60-Pad2)
- MX62 pad 2: Net-(D60-Pad2) -> COL0
- MX63 pad 1: COL1 -> Net-(D61-Pad2)
- MX63 pad 2: Net-(D61-Pad2) -> COL1
- MX64 pad 1: COL2 -> Net-(D62-Pad2)
- MX64 pad 2: Net-(D62-Pad2) -> COL2
- MX65 pad 1: COL6 -> Net-(D63-Pad2)
- MX65 pad 2: Net-(D63-Pad2) -> COL6
- MX66 pad 1: COL9 -> Net-(D64-Pad2)
- MX66 pad 2: Net-(D64-Pad2) -> COL9
- MX67 pad 1: COL10 -> Net-(D65-Pad2)
- MX67 pad 2: Net-(D65-Pad2) -> COL10
- MX68 pad 1: COL11 -> Net-(D66-Pad2)
- MX68 pad 2: Net-(D66-Pad2) -> COL11
- MX69 pad 1: COL12 -> Net-(D67-Pad2)
- MX69 pad 2: Net-(D67-Pad2) -> COL12
- MX7 pad 1: COL6 -> Net-(D7-Pad2)
- MX7 pad 2: Net-(D7-Pad2) -> COL6
- MX70 pad 1: COL13 -> Net-(D68-Pad2)
- MX70 pad 2: Net-(D68-Pad2) -> COL13
- MX71 pad 1: COL15 -> Net-(D69-Pad2)
- MX71 pad 2: Net-(D69-Pad2) -> COL15
- MX72 pad 1: COL9 -> Net-(D64-Pad2)
- MX72 pad 2: Net-(D64-Pad2) -> COL9
- MX73 pad 1: COL11 -> Net-(D66-Pad2)
- MX73 pad 2: Net-(D66-Pad2) -> COL11
- MX8 pad 1: COL7 -> Net-(D8-Pad2)
- MX8 pad 2: Net-(D8-Pad2) -> COL7
- MX9 pad 1: COL8 -> Net-(D9-Pad2)
- MX9 pad 2: Net-(D9-Pad2) -> COL8
- U2 pad 36: COL0 -> ROW2
- U2 pad 37: ROW2 -> COL0
- U2 pad 38: ROW3 -> ROW4
- U2 pad 39: COL2 -> ROW3
- U2 pad 40: ROW4 -> COL2
Routing:
- net COL2: track 215.9 -> 143.2 mm
- net ROW0: track 326.0 -> 276.9 mm
- net ROW3: track 340.1 -> 300.9 mm
- net Net-(D18-Pad2): track 11.6 -> 39.5 mm
- net ROW4: track 360.1 -> 333.6 mm
- net Net-(D16-Pad2): track 3.98 -> 29.4 mm
- net ROW2: track 325.9 -> 301.5 mm, vias 4 -> 2
- net MISO: track 74.9 -> 91.7 mm, vias 2 -> 0
- net +5V: track 106.5 -> 120.5 mm
- net SCK: track 72.7 -> 85.7 mm
- net MOSI: track 71.0 -> 83.2 mm
- net Net-(R4-Pad2): track 4.32 -> 14.6 mm
- net Net-(D19-Pad2): track 3.98 -> 14.2 mm
- net Net-(D46-Pad2): track 3.98 -> 12.9 mm
- net Net-(D20-Pad2): track 3.98 -> 12.9 mm
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
Commit message: Fix backspace key
Parts:
- moved D16 22.2 mm to (275.3, 5.87)
- moved MX17 19.1 mm to (254.6, 5.08)
- moved D15 15.7 mm to (272.1, 5.87)
Routing:
- net Net-(D16-Pad2): track 29.4 -> 5.23 mm
- net ROW0: track 276.9 -> 295.9 mm
- net Net-(D15-Pad2): track 15.9 -> 22.4 mm
- net COL15: track 358.0 -> 355.0 mm
Changed lines of the file:
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@@
     (thickness 1.6)
     (drawings 53)
-    (tracks 991)
+    (tracks 979)
     (zones 0)
     (modules 160)
@@
   )
   (module Diode_SMD:D_SOD-123 (layer B.Cu)
-    (at 253.0475 5.87375 90)
+    (at 275.2725 5.87375 90)
     (descr SOD-123)
     (tags SOD-123)
@@
   )
   (module Diode_SMD:D_SOD-123 (layer B.Cu)
-    (at 256.38125 5.87375 90)
+    (at 272.0975 5.87375 90)
     (descr SOD-123)
     (tags SOD-123)
@@
   )
   (module MX_Only:MXOnly-2U-NoLED (layer F.Cu)
-    (at 273.685 5.08)
+    (at 254.635 5.08)
     (fp_text reference MX17 (at 0 3.175) (layer Dwgs.User)
       (effects (font (size 1 1) (thickness 0.15)))
@@
   (segment (start 4.41375 2.54) (end 5.3975 3.52375) (width 0.25) (layer B.Cu) (net 4))
   (segment (start -6.35 2.54) (end 4.41375 2.54) (width 0.25) (layer B.Cu) (net 4))
-  (segment (start 256.2225 7.52375) (end 11.50625 7.52375) (width 0.25) (layer B.Cu) (net 5))
   (segment (start 11.50625 7.52375) (end 9.92625 7.52375) (width 0.25) (layer B.Cu) (net 5))
   (segment (start 9.92625 7.52375) (end 5.3975 7.52375) (width 0.25) (layer B.Cu) (net 5))
@@
   (segment (start 10.788065 26.645) (end 9.92 25.776935) (width 0.25) (layer F.Cu) (net 5))
   (segment (start 11.35375 26.645) (end 10.788065 26.645) (width 0.25) (layer F.Cu) (net 5))
+  (segment (start 11.50625 7.52375) (end 275.2725 7.52375) (width 0.25) (layer B.Cu) (net 5))
   (segment (start 8.5725 3.52375) (end 8.5725 4.22375) (width 0.25) (layer B.Cu) (net 6))
   (segment (start 9.55625 2.54) (end 8.5725 3.52375) (width 0.25) (layer B.Cu) (net 6))
@@
   (segment (start 236.56875 2.54) (end 235.585 3.52375) (width 0.25) (layer B.Cu) (net 18))
   (segment (start 241.3 2.54) (end 236.56875 2.54) (width 0.25) (layer B.Cu) (net 18))
-  (segment (start 269.875 2.54) (end 260.35 2.54) (width 0.25) (layer B.Cu) (net 19))
-  (segment (start 256.38125 4.22375) (end 256.38125 3.06516) (width 0.25) (layer B.Cu) (net 19))
-  (segment (start 258.1064 1.34001) (end 259.15001 1.34001) (width 0.25) (layer B.Cu) (net 19))
-  (segment (start 256.38125 3.06516) (end 258.1064 1.34001) (width 0.25) (layer B.Cu) (net 19))
-  (segment (start 259.15001 1.34001) (end 260.35 2.54) (width 0.25) (layer B.Cu) (net 19))
-  (segment (start 278.06 2.54) (end 279.4 2.54) (width 0.25) (layer B.Cu) (net 20))
-  (segment (start 274.78 0.89) (end 276.43 2.54) (width 0.25) (layer B.Cu) (net 20))
-  (segment (start 269.18 0.89) (end 274.78 0.89) (width 0.25) (layer B.Cu) (net 20))
-  (segment (start 254.58625 4.22375) (end 257.92 0.89) (width 0.25) (layer B.Cu) (net 20))
-  (segment (start 276.43 2.54) (end 278.06 2.54) (width 0.25) (layer B.Cu) (net 20))
-  (segment (start 257.92 0.89) (end 261.03 0.89) (width 0.25) (layer B.Cu) (net 20))
-  (segment (start 261.03 0.89) (end 262.22999 2.08999) (width 0.25) (layer B.Cu) (net 20))
-  (segment (start 253.0475 4.22375) (end 254.58625 4.22375) (width 0.25) (layer B.Cu) (net 20))
-  (segment (start 262.22999 2.08999) (end 267.98001 2.08999) (width 0.25) (layer B.Cu) (net 20))
-  (segment (start 267.98001 2.08999) (end 269.18 0.89) (width 0.25) (layer B.Cu) (net 20))
+  (segment (start 250.825 2.54) (end 260.35 2.54) (width 0.25) (layer B.Cu) (net 19))
+  (segment (start 272.0975 3.52375) (end 272.0975 4.22375) (width 0.25) (layer B.Cu) (net 19))
+  (segment (start 271.11375 2.54) (end 272.0975 3.52375) (width 0.25) (layer B.Cu) (net 19))
+  (segment (start 260.35 2.54) (end 271.11375 2.54) (width 0.25) (layer B.Cu) (net 19))
+  (segment (start 275.2725 3.52375) (end 275.2725 4.22375) (width 0.25) (layer B.Cu) (net 20))
+  (segment (start 276.25625 2.54) (end 275.2725 3.52375) (width 0.25) (layer B.Cu) (net 20))
+  (segment (start 279.4 2.54) (end 276.25625 2.54) (width 0.25) (layer B.Cu) (net 20))
   (segment (start -5.715 23.3675) (end -5.715 24.0675) (width 0.25) (layer B.Cu) (net 21))
   (segment (start -3.9375 21.59) (end -5.715 23.3675) (width 0.25) (layer B.Cu) (net 21))
@@
   (segment (start 266.7 6.59) (end 272.75 12.64) (width 0.25) (layer F.Cu) (net 99))
   (segment (start 266.7 0) (end 266.7 6.59) (width 0.25) (layer F.Cu) (net 99))
-  (segment (start 266.7 0) (end 268.29099 0) (width 0.25) (layer B.Cu) (net 99))
-  (segment (start 268.29099 0) (end 276.225 0) (width 0.25) (layer B.Cu) (net 99))
   (segment (start 272.75 44.87) (end 272.75 39.96) (width 0.25) (layer F.Cu) (net 99))
   (segment (start 272.75 39.96) (end 272.75 12.64) (width 0.25) (layer F.Cu) (net 99))
@@
   (segment (start 23.749989 44.785651) (end 23.749989 42.0136) (width 0.25) (layer B.Cu) (net 99))
   (segment (start 25.813098 46.84876) (end 23.749989 44.785651) (width 0.25) (layer B.Cu) (net 99))
+  (segment (start 257.175 0) (end 266.7 0) (width 0.25) (layer B.Cu) (net 99))
   (segment (start 285.75 18.85) (end 285.75 38.1) (width 0.25) (layer F.Cu) (net 100))
   (segment (start 285.75 38.1) (end 285.75 57.15) (width 0.25) (layer F.Cu) (net 100))
@@
   (segment (start 23.523752 34.63875) (end 25.20002 36.315018) (width 0.25) (layer B.Cu) (net 100))
   (segment (start 22.71375 34.63875) (end 23.523752 34.63875) (width 0.25) (layer B.Cu) (net 100))
-  (segment (start 285.75 0) (end 285.75 7.10375) (width 0.25) (layer F.Cu) (net 100))
-  (segment (start 285.75 7.10375) (end 282.20375 10.65) (width 0.25) (layer F.Cu) (net 100))
-  (segment (start 282.20375 15.50375) (end 285.75 19.05) (width 0.25) (layer F.Cu) (net 100))
-  (segment (start 282.20375 10.65) (end 282.20375 15.50375) (width 0.25) (layer F.Cu) (net 100))
+  (segment (start 285.75 19.05) (end 285.75 0) (width 0.25) (layer F.Cu) (net 100))
   (segment (start 18.28375 49.84444) (end 18.28375 51.0925) (width 0.25) (layer B.Cu) (net 101))
   (segment (start 13.01375 40.53875) (end 14.413714 41.938714) (width 0.25) (layer B.Cu) (net 101))
